File: Kicad-Weather-Station/Kicad-Weather-Station.sch (KiCad schematic (older format))
At the start: 63 parts, among them CON1 Solar Panel, J1 MicroSD, P1 CONN_01X25, P10 CONN_01X01, P11 CONN_01X01, P12 CONN_01X01, P2 CONN_01X25, P3 Rain Gauge, P4 Temperature/Humidity, P5 Wind Speed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

Commit message: Corrections to PCB schematic.
Parts:
- added JP2: JUMPER3, WeatherStation:PINHEAD1-3, symbol JUMPER3
- added unit 4 of U1
Connections:
- wire segments 68 -> 104
- no-connect marks 33 -> 34
Other:
- note added: "Battery\nVoltage"
- moved on the sheet: C4, C5, R22, R9, R?, U4

Commit message: Update schematic and PCB to allow some sensors to be powered off.
Parts:
- gave numbers to parts that had none: 1
Connections:
- wire segments 104 -> 69

Commit message: Clean up PCB footprints and generate gerbers.
Parts:
- RV1: footprint Potentiometers:Potentiometer_Bourns_3339P_Angular_ScrewUp -> WeatherStation:Potentiometer_Bourns_3339P_Angular_ScrewUp
Connections:
- no-connect marks 34 -> 35
Changed lines of the file:
@@
 F 0 "RV1" V 6500 2150 50  0000 C CNN
 F 1 "100K" V 6500 2400 50  0000 C CNN
-F 2 "Potentiometers:Potentiometer_Bourns_3339P_Angular_ScrewUp" H 6650 2350 50  0001 C CNN
+F 2 "WeatherStation:Potentiometer_Bourns_3339P_Angular_ScrewUp" H 6650 2350 50  0001 C CNN
 F 3 "" H 6650 2350 50  0000 C CNN
 	1    6650 2350
@@
 $Comp
 L PWR_FLAG #FLG029
-U 1 1 57978E15
-P 8450 1000
-F 0 "#FLG029" H 8450 1095 50  0001 C CNN
-F 1 "PWR_FLAG" H 8450 1180 50  0000 C CNN
-F 2 "" H 8450 1000 50  0000 C CNN
-F 3 "" H 8450 1000 50  0000 C CNN
-	1    8450 1000
-	1    0    0    -1
-$EndComp
-$Comp
-L Earth #PWR030
-U 1 1 57978FD5
-P 8450 1000
-F 0 "#PWR030" H 8450 750 50  0001 C CNN
-F 1 "Earth" H 8450 850 50  0001 C CNN
-F 2 "" H 8450 1000 50  0000 C CNN
-F 3 "" H 8450 1000 50  0000 C CNN
-	1    8450 1000
-	1    0    0    -1
-$EndComp
-$Comp
-L PWR_FLAG #FLG031
 U 1 1 5797995C
 P 9400 1500
-F 0 "#FLG031" H 9400 1595 50  0001 C CNN
+F 0 "#FLG029" H 9400 1595 50  0001 C CNN
 F 1 "PWR_FLAG" H 9400 1680 50  0000 C CNN
 F 2 "" H 9400 1500 50  0000 C CNN
@@
 PB15
 $Comp
-L Earth #PWR032
+L Earth #PWR030
 U 1 1 579905E5
 P 1850 7000
-F 0 "#PWR032" H 1850 6750 50  0001 C CNN
+F 0 "#PWR030" H 1850 6750 50  0001 C CNN
 F 1 "Earth" H 1850 6850 50  0001 C CNN
 F 2 "" H 1850 7000 50  0000 C CNN
@@
 $EndComp
 $Comp
-L Earth #PWR033
+L Earth #PWR031
 U 1 1 57990837
 P 2250 7000
-F 0 "#PWR033" H 2250 6750 50  0001 C CNN
+F 0 "#PWR031" H 2250 6750 50  0001 C CNN
 F 1 "Earth" H 2250 6850 50  0001 C CNN
 F 2 "" H 2250 7000 50  0000 C CNN
@@
 $EndComp
 $Comp
-L Earth #PWR034
+L Earth #PWR032
 U 1 1 579908DE
 P 2350 7000
-F 0 "#PWR034" H 2350 6750 50  0001 C CNN
+F 0 "#PWR032" H 2350 6750 50  0001 C CNN
 F 1 "Earth" H 2350 6850 50  0001 C CNN
 F 2 "" H 2350 7000 50  0000 C CNN
@@
 $EndComp
 $Comp
-L Earth #PWR035
+L Earth #PWR033
 U 1 1 57990985
 P 2450 7000
-F 0 "#PWR035" H 2450 6750 50  0001 C CNN
+F 0 "#PWR033" H 2450 6750 50  0001 C CNN
 F 1 "Earth" H 2450 6850 50  0001 C CNN
 F 2 "" H 2450 7000 50  0000 C CNN
@@
 $EndComp
 $Comp
-L Earth #PWR036
+L Earth #PWR034
 U 1 1 57990A2C
 P 2550 7000
-F 0 "#PWR036" H 2550 6750 50  0001 C CNN
+F 0 "#PWR034" H 2550 6750 50  0001 C CNN
 F 1 "Earth" H 2550 6850 50  0001 C CNN
 F 2 "" H 2550 7000 50  0000 C CNN
@@
 $EndComp
 $Comp
-L Earth #PWR037
+L Earth #PWR035
 U 1 1 5798550B
 P 8750 3800
-F 0 "#PWR037" H 8750 3550 50  0001 C CNN
+F 0 "#PWR035" H 8750 3550 50  0001 C CNN
 F 1 "Earth" H 8750 3650 50  0001 C CNN
 F 2 "" H 8750 3800 50  0000 C CNN
@@
 $EndComp
 $Comp
-L Earth #PWR038
+L Earth #PWR036
 U 1 1 579855CA
 P 8750 4050
-F 0 "#PWR038" H 8750 3800 50  0001 C CNN
+F 0 "#PWR036" H 8750 3800 50  0001 C CNN
 F 1 "Earth" H 8750 3900 50  0001 C CNN
 F 2 "" H 8750 4050 50  0000 C CNN
@@
 $EndComp
 $Comp
-L Earth #PWR039
+L Earth #PWR037
 U 1 1 57985689
 P 8750 4300
-F 0 "#PWR039" H 8750 4050 50  0001 C CNN
+F 0 "#PWR037" H 8750 4050 50  0001 C CNN
 F 1 "Earth" H 8750 4150 50  0001 C CNN
 F 2 "" H 8750 4300 50  0000 C CNN
@@
 $EndComp
 $Comp
-L Earth #PWR040
+L Earth #PWR038
 U 1 1 57985748
 P 8750 4600
-F 0 "#PWR040" H 8750 4350 50  0001 C CNN
+F 0 "#PWR038" H 8750 4350 50  0001 C CNN
 F 1 "Earth" H 8750 4450 50  0001 C CNN
 F 2 "" H 8750 4600 50  0000 C CNN
@@
 $EndComp
 $Comp
-L Earth #PWR041
+L Earth #PWR039
 U 1 1 57986899
 P 8750 4600
-F 0 "#PWR041" H 8750 4350 50  0001 C CNN
+F 0 "#PWR039" H 8750 4350 50  0001 C CNN
 F 1 "Earth" H 8750 4450 50  0001 C CNN
 F 2 "" H 8750 4600 50  0000 C CNN
@@
 $EndComp
 $Comp
-L Earth #PWR042
+L Earth #PWR040
 U 1 1 5798689F
 P 8750 4900
-F 0 "#PWR042" H 8750 4650 50  0001 C CNN
+F 0 "#PWR040" H 8750 4650 50  0001 C CNN
 F 1 "Earth" H 8750 4750 50  0001 C CNN
 F 2 "" H 8750 4900 50  0000 C CNN
@@
 $EndComp
 $Comp
-L Earth #PWR043
+L Earth #PWR041
 U 1 1 57C198FD
 P 2750 7000
-F 0 "#PWR043" H 2750 6750 50  0001 C CNN
+F 0 "#PWR041" H 2750 6750 50  0001 C CNN
 F 1 "Earth" H 2750 6850 50  0001 C CNN
 F 2 "" H 2750 7000 50  0000 C CNN
@@
 PD2
 $Comp
-L Earth #PWR044
+L Earth #PWR042
 U 1 1 59EB8994
 P 5700 4600
-F 0 "#PWR044" H 5700 4350 50  0001 C CNN
+F 0 "#PWR042" H 5700 4350 50  0001 C CNN
 F 1 "Earth" H 5700 4450 50  0001 C CNN
 F 2 "" H 5700 4600 50  0000 C CNN
@@
 Sensor Power\nEnable
 $Comp
-L Earth #PWR045
+L Earth #PWR043
 U 1 1 59EBCEAA
 P 5100 4600
-F 0 "#PWR045" H 5100 4350 50  0001 C CNN
+F 0 "#PWR043" H 5100 4350 50  0001 C CNN
 F 1 "Earth" H 5100 4450 50  0001 C CNN
 F 2 "" H 5100 4600 50  0000 C CNN
@@
 $EndComp
 $Comp
-L Earth #PWR046
+L Earth #PWR044
 U 1 1 59F0C357
 P 6200 4600
-F 0 "#PWR046" H 6200 4350 50  0001 C CNN
+F 0 "#PWR044" H 6200 4350 50  0001 C CNN
 F 1 "Earth" H 6200 4450 50  0001 C CNN
 F 2 "" H 6200 4600 50  0000 C CNN
@@
 $EndComp
 $Comp
-L Earth #PWR047
+L Earth #PWR045
 U 1 1 59F89224
 P 10000 6050
-F 0 "#PWR047" H 10000 5800 50  0001 C CNN
+F 0 "#PWR045" H 10000 5800 50  0001 C CNN
 F 1 "Earth" H 10000 5900 50  0001 C CNN
 F 2 "" H 10000 6050 50  0000 C CNN
@@
 	7850 1500 9400 1500
 $Comp
-L Earth #PWR048
+L Earth #PWR046
 U 1 1 5A067E16
 P 2800 1250
-F 0 "#PWR048" H 2800 1000 50  0001 C CNN
+F 0 "#PWR046" H 2800 1000 50  0001 C CNN
 F 1 "Earth" H 2800 1100 50  0001 C CNN
 F 2 "" H 2800 1250 50  0000 C CNN
@@
 	2800 1250 2800 1200
 $Comp
-L Earth #PWR049
+L Earth #PWR047
 U 1 1 5A06817B
 P 3100 1250
-F 0 "#PWR049" H 3100 1000 50  0001 C CNN
+F 0 "#PWR047" H 3100 1000 50  0001 C CNN
 F 1 "Earth" H 3100 1100 50  0001 C CNN
 F 2 "" H 3100 1250 50  0000 C CNN
@@
 	3100 1250 3100 1200
 $Comp
-L Earth #PWR050
+L Earth #PWR048
 U 1 1 5A0A7600
 P 10250 2150
-F 0 "#PWR050" H 10250 1900 50  0001 C CNN
+F 0 "#PWR048" H 10250 1900 50  0001 C CNN
 F 1 "Earth" H 10250 2000 50  0001 C CNN
 F 2 "" H 10250 2150 50  0000 C CNN
@@
 +3.3V-M
 $Comp
-L Earth #PWR?
+L Earth #PWR049
 U 1 1 5A430765
 P 10200 6050
-F 0 "#PWR?" H 10200 5800 50  0001 C CNN
+F 0 "#PWR049" H 10200 5800 50  0001 C CNN
 F 1 "Earth" H 10200 5900 50  0001 C CNN
 F 2 "" H 10200 6050 50  0000 C CNN
@@
 	1    0    0    -1
 $EndComp
+NoConn ~ 2900 5150
 $EndSCHEMATC

Commit message: Added missing inversion stage for battery charge MOSFET driver section. Removed clunky earth pin holes and added tracks with vias in the earthing part to ensure that all earths can be connected after zone fill.
Parts:
- removed P10, P11, P12, P8, P9: CONN_01X01, WeatherStation:SIL-1, symbol CONN_01X01
- added Q10: MMBT3904, WeatherStation:SOT23EBC, symbol Q_NPN_EBC
- R17: value 100K -> 10K
Connections:
- wire segments 69 -> 71
Other:
- moved on the sheet: Q4, Q5, Q6, Q7, Q8, R16, R9

Commit message: Second version of changes to fix MOSFET drivers. Use AND gate form of inverter to ensure that battery charge MOSFET is off when solar panel measurement is on. This does not need any transistors and is two resistors less.
Parts:
- removed Q10: MMBT3904, WeatherStation:SOT23EBC, symbol Q_NPN_EBC
- removed R17: 10K, WeatherStation:SM0603_Resistor, symbol R
- removed R7: 100K, WeatherStation:SM0603_Resistor, symbol R
Connections:
- wire segments 71 -> 99
Other:
- note added: "Charge\nEnable"
- note removed: "Charge\nDisable"
- moved on the sheet: Q2, Q3, Q4, Q5, Q6, R16, R2, R6, R9
